File: Hardware/KiCAD files/VECTRON_V1.kicad_sch (KiCad schematic)
At the start: 90 parts, among them J1 Screw_01x02, J2 Screw_01x02, J3 Screw_01x02, Q1 SIS447DN, U1 STM32F411CEUx, U2 TPS563201, U3 TPS563201, U4 AMS1117-3.3

Commit message: added bmp and magnetometer
Parts:
- removed C41, C42, C43, C44, C45, C46, C5, C6: C, symbol Device:C
- removed R15: 10k, symbol Device:R
- removed R21, R22, R5, R6: R, symbol Device:R
- removed U1: STM32F411CEUx, Package_DFN_QFN:QFN-48-1EP_7x7mm_P0.5mm_EP5.6x5.6mm, symbol MCU_ST_STM32F4:STM32F411CEUx
- added C10, C100, C101, C102, C103, C104, C105, C106, C107, C108, C109, C110, C111, C33, C34, C35, C36, C52, C53, C62, C63, C7, C77, C78, C8, C87, C88, C9, C98, C99: C, symbol Device:C
- added C112: 220nf, symbol Device:C
- added C113, C115, C21, C22, C23, C24, C25, C26, C29, C31, C32, C64, C65, C66, C72, C75, C79, C83, C86, C89, C95: 100nf, symbol Device:C
- added C114, C18, C19, C20, C30, C71, C73, C74, C76, C82, C84, C85, C90: 10uf, symbol Device:C
- added C48, C49, C50, C51: 10pf, symbol Device:C
- added C67, C68: 2u2f, symbol Device:C
- added C69, C70, C80, C81: 22uf, symbol Device:C
- added C96, C97: 100nf, Capacitor_SMD:C_0603_1608Metric, symbol Device:C
- added D10, D7, D8: SLESD5Z5C, symbol ESD_Diodes:ESD_DIODE
- added D11: PESD5V0U1BB, symbol ESD_Diodes:ESD_DIODE
- added D3: white, LED_SMD:LED_0603_1608Metric, symbol Device:LED
- added D4: WS2812B-2020, LED_SMD:LED_WS2812B-2020_PLCC4_2.0x2.0mm, symbol LED:WS2812B-2020
- added FB1: BLM18AG121SN1D, symbol Device:FerriteBead
- added J4: Conn_01x06_Pin, symbol Connector:Conn_01x06_Pin
- added J5: Conn_01x04_Pin, symbol Connector:Conn_01x04_Pin
- added J6, J7: USB_C_Receptacle_USB2.0_16P, symbol Connector:USB_C_Receptacle_USB2.0_16P
- added JP1, JP3, JP4: Jumper, Jumper:SolderJumper-2_P1.3mm_Open_RoundedPad1.0x1.5mm, symbol Jumper:SolderJumper_2_Open
- added JP2: Solder Jumper, symbol Jumper:SolderJumper_2_Open
- added L3, L4: SWPA5040S3R3NT 3u3h, Inductor_SMD:L_Sunlord_SWPA5040S, symbol Device:L
- added Q2: BSS123IXTSA1, Package_TO_SOT_SMD:SOT-23, symbol Transistor_FET:BSS123
- added R10, R16, R17, R26, R31, R32, R40, R41, R47, R48, R63, R64, R65, R66, R67, R68, R69, R7, R70, R71, R72, R73, R74, R75, R76, R9: R, symbol Device:R
- added R11, R12, R30, R33, R36, R45, R77: 10k, symbol Device:R
- added R18, R19: 0Ω, symbol Device:R
- added R27, R34, R42, R51, R52, R53, R54: 5k1, symbol Device:R
- added R35, R43: 54k9, symbol Device:R
- added R37: 1k, symbol Device:R
- added R38, R44, R46: 2k2, symbol Device:R
- added R39: 330, symbol Device:R
- added R56, R57, R59, R60: 22Ω, symbol Device:R
- added R61, R62: 100k, Resistor_SMD:R_0603_1608Metric, symbol Device:R
- added S1, S2: TSA017A2518B, digikey-footprints:Switch_Tactile_THT_B3F-1xxx, symbol dk_Tactile-Switches:B3F-1000
- added U1: LIS2MDL, Package_LGA:LGA-12_2x2mm_P0.5mm, symbol Sensor_Magnetic:LIS2MDL
- added U2: BMP280, Package_LGA:Bosch_LGA-8_2x2.5mm_P0.65mm_ClockwisePinNumbering, symbol Sensor_Pressure:BMP280
- added U4: ISM330DHCX, Package_LGA:LGA-14_3x2.5mm_P0.5mm_LayoutBorder3x4y, symbol Sensor_Motion:ISM330DHCX
- added U6: STM32F407VGTx, Package_QFP:LQFP-100_14x14mm_P0.5mm, symbol MCU_ST_STM32F4:STM32F407VGTx
- added U7, U8: TPS563201, Package_TO_SOT_SMD:SOT-23-6, symbol VECTRON_V1:TPS563201
- added Y1: 25MHz, symbol Device:Crystal_GND24
- added Y2: 32.678KHz, symbol Device:Crystal
- C27: value C -> 100nf
- C28: value C -> 10uf
- R15: renamed from R7; value 1k -> 2k2
- R20: value R -> 5k1
- R23, R24: value R -> 10M
- R49: renamed from R18; value 1k -> 560
- R58: renamed from R19; value 1k -> 750
- R8: value 10k -> R
- renumbered C7 to C11, C8 to C12, C9 to C13, C10 to C14, C11 to C15, C12 to C16, C13 to C17, C14 to C37, C15 to C38, C16 to C39, C17 to C40, C18 to C41, C19 to C42, C20 to C43, C21 to C44, C22 to C45, C23 to C46, C24 to C47, C25 to C5, C29 to C54, C30 to C55, C31 to C56, C32 to C57, C33 to C58, C34 to C59, C26 to C6, C35 to C60, C36 to C61, C37 to C91, C38 to C92, C39 to C93, C40 to C94, D5 to D12, D3 to D5, D4 to D6, D6 to D9, R9 to R21, R10 to R22, R16 to R28, R17 to R29, R11 to R5, R26 to R50, R27 to R55, R12 to R6, U2 to U3, U3 to U5, U4 to U9
Connections:
- net +3V3: now also C113.2, C114.2, C115.2, C20.2, C21.2, C22.2, C23.2, C24.2, C25.2, C26.2, C29.2, C30.2, C31.2, C32.2, FB1.2, J4.6 (Pin_6), J5.4 (Pin_4), JP1.2 (B), Q2.1 (G), R11.2, R30.1, R44.1, R46.1, R77.2, S2.3, S2.4, U1.10 (Vdd_IO), U1.9 (Vdd), U2.6 (VDDIO), U2.8 (VDD), U6.100 (VDD), U6.11 (VDD), U6.19 (VDD), U6.28 (VDD), U6.50 (VDD), U6.75 (VDD)
- net +5V: now also C76.2, D4.4 (VDD), R38.1
- net +VCOM: now also R20.1, C73.2, C74.2, C75.2, C84.2, C85.2, C86.2, R27.1, R34.1, R42.1, U7.3 (VIN), U8.3 (VIN); no longer R8.1
- net +VUSB: now also C89.2, C90.2, D7.2, J6.A4 (VBUS), J6.A9 (VBUS), J6.B4 (VBUS), J6.B9 (VBUS)
- net EN3: now also R27.2
- net EN5: now also R20.2, R34.2, R42.2, U7.5 (EN), U8.5 (EN); no longer R8.2
- net GND: now also C27.1, C28.1, D9.1, C112.1, C113.1, C114.1, C115.1, C18.1, C19.1, C20.1, C21.1, C22.1, C23.1, C24.1, C25.1, C26.1, C29.1, C30.1, C31.1, C32.1, C48.1, C49.1, C50.1, C51.1, C64.2, C65.1, C67.1, C68.1, C69.1, C70.1, C71.1, C72.1, C73.1, C74.1, C75.1, C76.1, C80.1, C81.1, C82.1, C83.1, C84.1, C85.1, C86.1, C89.1, C90.1, C95.1, C96.2, C97.2, D10.1, D11.1, D3.1 (K), D4.2 (VSS), D7.1, D8.1, J4.4 (Pin_4), J5.2 (Pin_2), J6.A1 (GND), J6.A12 (GND), J6.B1 (GND), J6.B12 (GND), J7.A1 (GND), J7.A12 (GND), J7.B1 (GND), J7.B12 (GND), JP3.2 (B), JP4.2 (B), R12.2, R33.2, R36.2, R45.2, R51.2, R52.2, R53.2, R54.2, R61.2, R62.2, S1.3, S1.4, U1.6 (GND), U1.8 (GND), U2.1 (GND), U2.7 (GND), U6.10 (VSS), U6.20 (VSSA), U6.27 (VSS), U6.74 (VSS), U6.99 (VSS), U7.1 (GND), U8.1 (GND), Y1.2, Y1.4
- net SW5: now also C66.2, C79.2, L3.1, L4.1, U7.2 (SW), U8.2 (SW)
- net VBST5: now also C66.1, C79.1, U7.6 (VBST), U8.6 (VBST)
- net VFB5: now also R35.2, R36.1, R43.2, R45.1, U7.4 (VFB), U8.4 (VFB)
- net +3V3A: now reaches C28.2
- net +3V3A: now also C27.2, FB1.1, U6.21 (VREF+), U6.22 (VDDA)
- net LSE_IN: now reaches R24.1
- net LSE_IN: now also C50.2, U6.7 (PC13), Y2.1
- net LSE_OUT: now reaches R24.2
- net LSE_OUT: now also C51.2, U6.8 (PC14), Y2.2
- net MAIN_BAT: now reaches R50.2, R55.1
- net MAIN_BAT: now also C95.2
- net HSE_OUT: now reaches R23.1
- net HSE_OUT: now also C48.2, U6.13 (PH1), Y1.1
- net HSE_IN: now reaches R23.2
- net HSE_IN: now also C49.2, U6.12 (PH0), Y1.3
- net USB_FS_D-: now reaches D9.2
- net USB_FS_D-: now also J7.A7 (D-), J7.B7 (D-), R57.1
- net +EMGR_BAT renamed +COIN_BAT
- net +COIN_BAT: now also C18.2, C19.2, U6.6 (VBAT)
- new net: Q2.3 (D), R38.2, R39.1
- new net: D4.3 (DIN), R39.2
- new net: J5.1 (Pin_1), R19.2
- new net: J5.3 (Pin_3), R18.2
- new net: U4.6 (GND), U4.7 (GND)
- new net: J4.2 (Pin_2), JP2.2 (B)
- new net: C112.2, U1.5 (C1)
- new net: J7.A4 (VBUS), J7.A9 (VBUS), J7.B4 (VBUS), J7.B9 (VBUS)
- new net +5VS1: C69.2, C70.2, C71.2, C72.2, L3.2, R35.1
- new net +5VS2: C80.2, C81.2, C82.2, C83.2, L4.2, R43.1
- new net BMP_CSB: R11.1, U2.2 (CSB)
- new net BMP_SDO: JP1.1 (A), R12.1, U2.5 (SDO)
- new net BOOT: C65.2, R33.1, S2.1, S2.2, U6.94 (BOOT0)
- new net CC1FS: J7.A5 (CC1), R52.1
- new net CC1HS: J6.A5 (CC1), R51.1
- new net CC2FS: J7.B5 (CC2), R54.1
- new net CC2HS: J6.B5 (CC2), R53.1
- new net FS_D+: R60.2
- new net FS_D-: R57.2
- new net HS_D+: R59.2
- new net HS_D-: R56.2
- new net I2C1_SCL: R46.2, U1.1 (SCL/SPC), U2.4 (SCK)
- new net I2C1_SDA: R44.2, U1.4 (SDA/SDI/SDO), U2.3 (SDI)
- new net LIS_CS: R77.1, U1.3 (~{CS})
- new net NRST: C64.1, JP2.1 (A), R30.2, S1.1, S1.2, U6.14 (NRST)
- new net PROG_LED: Q2.2 (S)
- new net SHIELD_FS: C97.1, J7.S1 (SHIELD), JP4.1 (A), R62.1
- new net SHIELD_HS: C96.1, J6.S1 (SHIELD), JP3.1 (A), R61.1
- new net STATUS_LED: R37.1
- new net STM_LED: D3.2 (A), R37.2
- new net SWCLK: J4.5 (Pin_5)
- new net SWDIO: J4.3 (Pin_3)
- new net SWO: J4.1 (Pin_1)
- new net USART1_RX: R18.1
- new net USART1_TX: R19.1
- new net USB_FS_D+: D11.2, J7.A6 (D+), J7.B6 (D+), R60.1
- new net USB_HS_D+: D10.2, J6.A6 (D+), J6.B6 (D+), R59.1
- new net USB_HS_D-: D8.2, J6.A7 (D-), J6.B7 (D-), R56.1
- new net VCAP_1: C67.2, U6.49 (VCAP_1)
- new net VCAP_2: C68.2, U6.73 (VCAP_2)
- no-connect marks 2 -> 9
Other:
- note added: "ANALOG FILTERING"
- note added: "BMP280 BAROMETER"
- note added: "BOOT TACTILE SWITCH"
- note added: "BUILT-IN LED"
- note added: "COIN CELL DECOUPLING CAPAS"
- note added: "DECOUPLING CAPS"
- note added: "HSE CRYSTAL"
- note added: "I2C ADDRESS SWITCHING"
- note added: "I2C PULL UP RESISTOR"
- note added: "LIS2MDL MAGNETOMETER"
- note added: "LSE CRYSTAL"
- note added: "MAIN DECOUPLING CAPS"
- note added: "POWER FLAGS"
- note added: "PROGRAMABLE RGB LED"
- note added: "RESET TACTILE SWITCH"
- note added: "ST-LINK DEBUGGER AND FLASHING"
- note added: "STM32"
- note added: "UART DEBUG AND FLASHING"
- note added: "USB DECOUPLING CAPS"
- note added: "USB ESD DIODES"
- note added: "USB TYPE C FULL SPEED"
- note added: "USB TYPE C HIGH SPEED"
- moved on the sheet: C5, C6, C91, C92, C93, C94, D12, D5, D6, D9, R49, R5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

Commit message: all connections made rechecking needed
Parts:
- removed C32: 100nf, symbol Device:C
- removed D12: SLESD5Z5C, symbol ESD_Diodes:ESD_DIODE
- added BZ1: CL8530A-CLDZ, Buzzer_Beeper:MagneticBuzzer_PUI_AT-0927-TT-6-R, symbol Device:Buzzer
- added C104, C110, C35, C54, C73, C77, C90: 10uf, symbol Device:C
- added C109, C45, C56, C64, C78, C92: 100nf, symbol Device:C
- added C44, C55, C63, C91: 10uf, Capacitor_SMD:C_0603_1608Metric, symbol Device:C
- added D10: PESD5V0U1BB, symbol ESD_Diodes:ESD_DIODE
- added D2: SS24-SMB, symbol Device:D_Schottky
- added D4: white, LED_SMD:LED_0603_1608Metric, symbol Device:LED
- added J6: GPS_ANT, digikey-footprints:Molex_734120114_UMC_RF_CONN_Vertical, symbol dk_Coaxial-Connectors-RF:0734120114
- added J7: Micro_SD_Card, symbol Connector:Micro_SD_Card
- added L2: 27nh, Inductor_SMD:L_0402_1005Metric, symbol Device:L
- added Q2: IRLML2502, symbol Simulation_SPICE:NMOS
- added R20: 1k, symbol Device:R
- added R27, R28, R39, R40, R41, R42, R43, R44, R45, R90, R91, R92, R93, R94, R95: 10k, symbol Device:R
- added R31, R38: 10Ω, symbol Device:R
- added U4: NEO-6M-GPS, NEO-6M-GPS:XCVR_NEO-6M-GPS, symbol NEO-6M-GPS:NEO-6M-GPS
- added U6: W25Q128JVS, Package_SO:SOIC-8_5.3x5.3mm_P1.27mm, symbol Memory_Flash:W25Q128JVS
- renumbered C83 to C100, C84 to C101, C85 to C102, C86 to C103, C87 to C105, C88 to C106, C89 to C107, C90 to C108, C91 to C111, C92 to C112, C93 to C113, C94 to C114, C95 to C115, C96 to C116, C97 to C117, C98 to C118, C99 to C119, C100 to C120, C101 to C121, C102 to C122, C103 to C123, C104 to C124, C105 to C125, C106 to C126, C107 to C127, C108 to C128, C109 to C129, C110 to C130, C111 to C131, C113 to C31, C114 to C32, C115 to C33, C31 to C34, C112 to C36, C33 to C37, C34 to C38, C35 to C39, C36 to C40, C37 to C41, C38 to C42, C39 to C43, C40 to C46, C41 to C47, C42 to C48, C43 to C49, C44 to C50, C45 to C51, C46 to C52, C47 to C53, C48 to C57, C49 to C58, C50 to C59, C51 to C60, C52 to C61, C53 to C62, C54 to C65, C55 to C66, C56 to C67, C57 to C68, C58 to C69, C59 to C70, C60 to C71, C61 to C72, C62 to C74, C63 to C75, C64 to C76, C65 to C79, C66 to C80, C67 to C81, C68 to C82, C69 to C83, C70 to C84, C71 to C85, C72 to C86, C73 to C87, C74 to C88, C75 to C89, C76 to C93, C77 to C94, C78 to C95, C79 to C96, C80 to C97, C81 to C98, C82 to C99, D8 to D11, D9 to D12, D10 to D13, D11 to D14, D2 to D3, D3 to D5, D4 to D6, D5 to D7, D6 to D8, D7 to D9, J6 to J8, J7 to J9, L2 to L3, L3 to L4, L4 to L5, Q2 to Q3, R77 to R11, R11 to R12, R12 to R13, R13 to R14, R14 to R15, R15 to R16, R16 to R17, R17 to R18, R18 to R19, R19 to R21, R20 to R22, R21 to R23, R22 to R24, R23 to R25, R24 to R26, R25 to R29, R26 to R30, R27 to R32, R28 to R33, R29 to R34, R30 to R35, R31 to R36, R32 to R37, R33 to R46, R34 to R47, R35 to R48, R36 to R49, R37 to R50, R38 to R51, R39 to R52, R40 to R53, R41 to R54, R42 to R55, R43 to R56, R44 to R57, R45 to R58, R46 to R59, R47 to R60, R48 to R61, R49 to R62, R50 to R63, R51 to R64, R52 to R65, R53 to R66, R54 to R67, R55 to R68, R56 to R69, R57 to R70, R58 to R71, R59 to R72, R60 to R73, R61 to R74, R62 to R75, R63 to R76, R64 to R77, R65 to R78, R66 to R79, R67 to R80, R68 to R81, R69 to R82, R70 to R83, R71 to R84, R72 to R85, R73 to R86, R74 to R87, R75 to R88, R76 to R89, U8 to U10, U9 to U11, U4 to U3, U3 to U5, U5 to U7, U6 to U8, U7 to U9
Connections:
- net +3V3: now also U3.5 (VDDIO), U3.8 (VDD), BZ1.1 (+), C35.2, C44.2, C45.2, C55.2, C56.2, C63.2, C64.2, C77.2, C78.2, C91.2, C92.2, J7.4 (VDD), R27.1, R28.1, R39.1, R40.1, R41.1, R42.1, R43.1, R44.1, R90.1, R91.1, R92.1, R93.1, R94.1, R95.1, U4.23 (VCC), U6.3 (~{WP}/IO_{2}), U6.7 (~{HOLD}/~{RESET}/IO_{3}), U6.8 (VCC)
- net +COIN_BAT: now also U4.22 (V_BCKP)
- net +VCOM: now also C104.2, C54.2, C73.2, C90.2, D2.1 (K)
- net EN5: no longer R47.2, R55.2, U10.5 (EN), U9.5 (EN)
- net GND: now also U3.2 (SDx), U3.3 (SCx), U3.6 (GND), U3.7 (GND), C104.1, C109.1, C110.1, C35.1, C44.1, C45.1, C54.1, C55.1, C56.1, C63.1, C64.1, C73.1, C77.1, C78.1, C90.1, C91.1, C92.1, D10.1, D4.1 (K), J6.1, J7.6 (VSS), J7.9 (SHIELD), Q2.3 (S), R45.2, U4.10 (GND), U4.12 (GND), U4.13 (GND), U4.24 (GND), U6.4 (GND)
- net SW5: no longer C80.2, C96.2, L4.1, L5.1, U10.2 (SW), U9.2 (SW)
- net USART2_RX: now also U4.20 (TXD1)
- net USART2_TX: now also U4.21 (RXD1)
- net VBST5: no longer C80.1, C96.1, U10.6 (VBST), U9.6 (VBST)
- net VFB5: no longer R48.2, R49.1, R56.2, R58.1, U10.4 (VFB), U9.4 (VFB)
- net SPI1_MISO: now reaches U3.1 (SDO/SA0)
- net SPI1_MISO: now also R93.2
- net IMU_CS: now reaches U3.12 (CS)
- net IMU_CS: now also R95.2
- net SPI1_SCK: now reaches U3.13 (SCL)
- net SPI1_SCK: now also R94.2
- net SPI1_MOSI: now reaches U3.14 (SDA)
- net SPI1_MOSI: now also R92.2
- net IMU_INT1: now reaches U3.4 (INT1)
- net IMU_INT2: now reaches U3.9 (INT2)
- net +VUSB_FS: now reaches J9.A4 (VBUS), J9.A9 (VBUS), J9.B4 (VBUS), J9.B9 (VBUS)
- net +VUSB_FS: now also C109.2, C110.2, D10.2, D2.2 (A)
- net +VUSB renamed +VUSB_HS
- new net: BZ1.2 (-), Q2.1 (D)
- new net BUZZER: R38.1
- new net BUZZ_GATE: Q2.2 (G), R38.2, R45.1
- new net ENS1: R47.2, U9.5 (EN)
- new net ENS2: R55.2, U10.5 (EN)
- new net RF_IN: J6.2, L2.2, U4.11 (RF_IN)
- new net SDIO_CK: J7.5 (CLK), R41.2
- new net SDIO_CMD: J7.3 (CMD), R42.2
- new net SDIO_D0: J7.7 (DAT0), R40.2
- new net SDIO_D1: J7.8 (DAT1), R39.2
- new net SDIO_D2: J7.1 (DAT2), R44.2
- new net SDIO_D3: J7.2 (DAT3/CD), R43.2
- new net SPI2_MISO: R91.2, U6.2 (DO/IO_{1})
- new net SPI2_MOSI: R90.2, U6.5 (DI/IO_{0})
- new net SPI2_SCK: R27.2, U6.6 (CLK)
- new net SPI_FLASH_CS: R28.2, U6.1 (~{CS})
- new net SWS1: C80.2, L4.1, U9.2 (SW)
- new net SWS2: C96.2, L5.1, U10.2 (SW)
- new net VBSTS1: C80.1, U9.6 (VBST)
- new net VBSTS2: C96.1, U10.6 (VBST)
- new net VCC_RF: R31.1, U4.8 (RSVD_8), U4.9 (VCC_RF)
- new net VFBS1: R48.2, R49.1, U9.4 (VFB)
- new net VFBS2: R56.2, R58.1, U10.4 (VFB)
- new net gps_inductor: L2.1, R31.2
- new net gps_led: D4.2 (A), R20.2
- new net gps_pulse: R20.1, U4.3 (TIMEPULSE)
- no-connect marks 9 -> 20
Other:
- note added: "ANTENNA"
- note added: "BUZZER"
- note added: "DECOUPLING CAPACITORS"
- note added: "ISM330DHCX IMU"
- note added: "MICRO SD CARD"
- note added: "NEO-6M GPS"
- note added: "W25Q128JVSIQ SPI FLASH"
- moved on the sheet: C41, C42, C43, D1, D6, Q3, R22, R32, R47, R51, R52, R55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

Commit message: finished according to me :)
Parts:
- removed C116, C117: 100nf, Capacitor_SMD:C_0603_1608Metric, symbol Device:C
- removed C66, C83, C84, C97, C98: 22uf, symbol Device:C
- removed C99: 10uf, symbol Device:C
- removed R19, R21: 0Ω, symbol Device:R
- removed R74, R75: 100k, Resistor_SMD:R_0603_1608Metric, symbol Device:R
- added C105, C112, C120, C121: 100nf, symbol Device:C
- added C106, C111, C51, C74, C75, C91, C92, C93: 10uf, symbol Device:C
- added J10, J11, J12, J13, J8, J9: 1X3-JST-XH, Connector_JST:JST_XH_B3B-XH-A_1x03_P2.50mm_Vertical, symbol Connector:Conn_01x03_Pin
- added J14: 01x03_Pin, symbol Connector:Conn_01x03_Pin
- added J15, J16, J20: 01x04_Pin, symbol Connector:Conn_01x04_Pin
- added J17: 1X4-JST-XH, symbol Connector:Conn_01x04_Pin
- added JP3, JP4: Jumper, Jumper:SolderJumper-2_P1.3mm_Open_RoundedPad1.0x1.5mm, symbol Jumper:SolderJumper_2_Open
- added R100, R99: 100k, symbol Device:R
- added R17, R18, R80: 10k, symbol Device:R
- added R25, R27, R30, R31, R32, R42, R48, R49, R54, R63, R64, R66, R69, R70: 10Ω, symbol Device:R_Small
- added R26, R29, R85, R90: 0Ω, symbol Device:R_Small
- C100, C103, C107, C50, C69, C86, C89: value 100nf -> 10uf
- C47, C48, C67: value 22uf -> 10uf
- C90: value 10uf -> 100nf
- J5: value Conn_01x04_Pin -> 1X4-JST-XH
- JP2: value Solder Jumper -> Jumper; footprint (none) -> Jumper:SolderJumper-2_P1.3mm_Open_RoundedPad1.0x1.5mm
- renumbered C105 to C109, C106 to C110, C110 to C113, C109 to C114, C111 to C115, C112 to C116, C113 to C117, C114 to C118, C115 to C119, C118 to C122, C119 to C123, C120 to C124, C121 to C125, C122 to C126, C123 to C127, C124 to C128, C125 to C129, C126 to C130, C127 to C131, C128 to C132, C129 to C133, C130 to C134, C131 to C135, C53 to C52, C52 to C53, C51 to C54, C54 to C55, C55 to C56, C56 to C57, C57 to C58, C58 to C59, C59 to C60, C60 to C61, C61 to C62, C62 to C63, C63 to C64, C64 to C65, C65 to C66, C74 to C76, C75 to C77, C76 to C78, C77 to C79, C78 to C80, C79 to C81, C80 to C82, C81 to C83, C82 to C84, C91 to C94, C92 to C95, C93 to C96, C94 to C97, C95 to C98, C96 to C99, J8 to J18, J9 to J19, JP3 to JP5, JP4 to JP6, R76 to R101, R77 to R102, R78 to R103, R79 to R104, R80 to R105, R81 to R106, R82 to R107, R83 to R108, R84 to R109, R85 to R110, R86 to R111, R87 to R112, R88 to R113, R89 to R114, R92 to R19, R93 to R20, R94 to R21, R95 to R22, R17 to R23, R18 to R24, R20 to R28, R22 to R33, R23 to R34, R24 to R35, R25 to R36, R26 to R37, R28 to R38, R27 to R39, R90 to R40, R91 to R41, R29 to R43, R30 to R44, R31 to R45, R32 to R46, R33 to R47, R34 to R50, R35 to R51, R36 to R52, R37 to R53, R38 to R55, R39 to R56, R40 to R57, R41 to R58, R42 to R59, R43 to R60, R44 to R61, R45 to R62, R46 to R65, R47 to R67, R48 to R68, R49 to R71, R50 to R72, R51 to R73, R52 to R74, R53 to R75, R54 to R76, R55 to R77, R56 to R78, R57 to R79, R58 to R81, R59 to R82, R60 to R83, R61 to R84, R62 to R86, R63 to R87, R64 to R88, R65 to R89, R66 to R91, R67 to R92, R68 to R93, R69 to R94, R70 to R95, R71 to R96, R72 to R97, R73 to R98
Connections:
- net +3V3: now also C70.2, C71.2, JP2.1 (A), J11.1 (Pin_1), JP4.2 (B), R17.1, R18.1; no longer J4.6 (Pin_6)
- net +5V: now also C51.2, J17.4 (Pin_4)
- net +5VS1: now also C87.2, C88.2, C89.2
- net +5VS2: now also C101.2, C102.2, C103.2, C104.2
- net +VCOM: now also C107.2, C108.2, C105.2, C106.2, C74.2, C75.2, C91.2, C92.2, C93.2; no longer C101.2, C102.2, C103.2, C104.2, C70.2, C71.2, C87.2, C88.2, C89.2
- net +VUSB_HS: now also C111.2, C112.2; no longer C107.2, C108.2
- net BUZZER: now also U8.35 (PB0)
- net FS_D+: now also U8.71 (PA12)
- net FS_D-: now also U8.70 (PA11)
- net GND: now also C105.1, C106.1, C111.1, C112.1, C120.2, C121.2, C51.1, C74.1, C75.1, C91.1, C92.1, C93.1, J10.3 (Pin_3), J11.3 (Pin_3), J12.3 (Pin_3), J13.3 (Pin_3), J14.1 (Pin_1), J15.1 (Pin_1), J16.1 (Pin_1), J17.2 (Pin_2), J20.1 (Pin_1), J8.3 (Pin_3), J9.3 (Pin_3), R100.2, R80.2, R99.2
- net HS_D+: now also U8.54 (PB15)
- net HS_D-: now also U8.53 (PB14)
- net I2C1_SCL: now also U8.95 (PB8), J14.3 (Pin_3)
- net I2C1_SDA: now also U8.96 (PB9), J14.2 (Pin_2)
- net IMU_CS: now also R19.2; no longer R22.2
- net IMU_INT1: now also U8.3 (PE4), R18.2, R27.1; no longer U3.4 (INT1)
- net IMU_INT2: now also U8.4 (PE5), R17.2, R30.1; no longer U3.9 (INT2)
- net LSE_IN: now also U8.8 (PC14); no longer U8.7 (PC13)
- net LSE_OUT: now also U8.9 (PC15); no longer U8.8 (PC14)
- net MAIN_BAT: now also U8.15 (PC0)
- net NRST: now also JP3.1 (A); no longer JP2.1 (A)
- net PROG_LED: now also U8.36 (PB1)
- net SDIO_CK: now also R70.2
- net SDIO_CMD: now also R49.1
- net SDIO_D0: now also R63.2
- net SDIO_D1: now also R64.2
- net SDIO_D2: now also R66.2
- net SDIO_D3: now also R69.2
- net SHIELD_FS: now also C121.1, R100.1
- net SHIELD_HS: now also C120.1, R99.1
- net SPI1_MISO: now also R21.2, U8.31 (PA6), J15.3 (Pin_3), R25.1; no longer R20.2, U3.1 (SDO/SA0)
- net SPI1_MOSI: now also R22.2, J15.4 (Pin_4), R32.2; no longer R19.2
- net SPI1_SCK: now also R20.2, J15.2 (Pin_2), R31.2; no longer R21.2
- net SPI2_MISO: now also R38.2, U8.17 (PC2), J16.3 (Pin_3), R42.1; no longer R41.2, U6.2 (DO/IO_{1})
- net SPI2_MOSI: now also R39.2, J16.4 (Pin_4), R54.2; no longer R40.2
- net SPI2_SCK: now also R40.2, J16.2 (Pin_2), R48.2; no longer R39.2
- net STATUS_LED: now also U8.59 (PD12)
- net SWCLK: now also U8.76 (PA14)
- net SWDIO: now also U8.72 (PA13)
- net SWO: now also U8.89 (PB3)
- net USART1_RX: now also U8.93 (PB7), R26.1
- net USART1_TX: now also U8.92 (PB6), R29.1
- net USART2_RX: now also U8.87 (PD6), R90.1
- net USART2_TX: now also U8.86 (PD5), R85.1
- net at U8.18 (PC3): now also R54.1
- net SERVO_X1: now reaches U8.23 (PA0)
- net SERVO_X1: now also J8.2 (Pin_2)
- net SERVO_X2: now reaches U8.24 (PA1)
- net SERVO_X2: now also J9.2 (Pin_2)
- net SERVO_Y1: now reaches U8.25 (PA2)
- net SERVO_Y1: now also J10.2 (Pin_2)
- net SERVO_Y2: now reaches U8.26 (PA3)
- net SERVO_Y2: now also J11.2 (Pin_2)
- net at U8.30 (PA5): now also R31.1
- net at U8.32 (PA7): now also R32.1
- net BOOT1: now reaches U8.37 (PB2)
- net BOOT1: now also JP4.1 (A), R80.1
- net at U8.47 (PB10): now also R48.1
- net RECOV_1: now reaches U8.63 (PC6)
- net RECOV_1: now also J12.2 (Pin_2)
- net RECOV_2: now reaches U8.64 (PC7)
- net RECOV_2: now also J13.2 (Pin_2)
- net at U8.65 (PC8): now also R63.1
- net at U8.66 (PC9): now also R64.1
- net at U8.78 (PC10): now also R66.1
- net at U8.79 (PC11): now also R69.1
- net at U8.80 (PC12): now also R70.1
- net at U8.83 (PD2): now also R49.2
- net at J5.1 (Pin_1): now also R29.2
- net at J5.3 (Pin_3): now also R26.2
- net at J4.2 (Pin_2): now also JP3.2 (B); no longer JP2.2 (B)
- net BOOT renamed BOOT0
- net SPI_FLASH_CS renamed FLASH_CS
- net FLASH_CS: now also R41.2; no longer R38.2
- new net: R27.2, U3.4 (INT1)
- new net: R25.2, U3.1 (SDO/SA0)
- new net: R30.2, U3.9 (INT2)
- new net: J4.6 (Pin_6), JP2.2 (B)
- new net: J17.3 (Pin_3), R85.2
- new net: J17.1 (Pin_1), R90.2
- new net: R42.2, U6.2 (DO/IO_{1})
Other:
- note added: "3V3 LDO (REDUNDANT)"
- note added: "BOOT1 SELECTOR"
- note added: "BUCK CONVERTER 3V3"
- note added: "FIN SERVO X1"
- note added: "FIN SERVO X2"
- note added: "FIN SERVO Y1"
- note added: "FIN SERVO Y2"
- note added: "FIN SERVOS"
- note added: "GPS DEBUGGING"
- note added: "I2C DEBUGGING"
- note added: "IMU DEBUGGING"
- note added: "RECOVERY SERVO 1"
- note added: "RECOVERY SERVO 2"
- note added: "RECOVERY SERVOS"
- note added: "SPI DEBUGGING"
- note added: "SPI FLASH DEBUGGING"
- note added: "STM32F407VGT6"
- note added: "XY117B-3.81"
- note removed: "(REDUNDANT)"
- note removed: "3V3 LDO"
- moved on the sheet: C113, C114, C44, C45, C49, C52, C53, C54, C55, C64, C65, C83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

Commit message: tiny changes
Parts:
- removed C1, C10, C109, C110, C122, C123, C124, C125, C126, C127, C128, C129, C130, C131, C132, C133, C134, C135, C2, C3, C37, C38, C39, C4, C40, C5, C6, C62, C63, C7, C76, C77, C8, C9, C97, C98: C, symbol Device:C
- removed J20: 01x04_Pin, symbol Connector:Conn_01x04_Pin
- removed J6: GPS_ANT, digikey-footprints:Molex_734120114_UMC_RF_CONN_Vertical, symbol dk_Coaxial-Connectors-RF:0734120114
- removed R1, R10, R101, R102, R103, R104, R105, R106, R107, R108, R109, R110, R111, R112, R113, R114, R14, R15, R2, R23, R24, R3, R4, R43, R44, R5, R52, R53, R6, R7, R75, R76, R8, R83, R84, R9: R, symbol Device:R
- added J6: U_FL-R-SMT, SparkFun-Connector:RP-SMA_Edge, symbol dk_Coaxial-Connectors-RF:U_FL-R-SMT_10_
- renumbered C11 to C1, C20 to C10, C21 to C11, C22 to C12, C23 to C13, C24 to C14, C25 to C15, C26 to C16, C27 to C17, C28 to C18, C29 to C19, C12 to C2, C30 to C20, C31 to C21, C32 to C22, C33 to C23, C34 to C24, C35 to C25, C36 to C26, C41 to C27, C42 to C28, C43 to C29, C13 to C3, C44 to C30, C45 to C31, C46 to C32, C47 to C33, C48 to C34, C49 to C35, C50 to C36, C51 to C37, C52 to C38, C53 to C39, C14 to C4, C54 to C40, C55 to C41, C56 to C42, C57 to C43, C58 to C44, C59 to C45, C60 to C46, C61 to C47, C64 to C48, C65 to C49, C15 to C5, C66 to C50, C67 to C51, C68 to C52, C69 to C53, C70 to C54, C71 to C55, C72 to C56, C73 to C57, C74 to C58, C75 to C59, C16 to C6, C78 to C60, C79 to C61, C80 to C62, C81 to C63, C82 to C64, C83 to C65, C84 to C66, C85 to C67, C86 to C68, C87 to C69, C17 to C7, C88 to C70, C89 to C71, C90 to C72, C91 to C73, C92 to C74, C93 to C75, C94 to C76, C95 to C77, C96 to C78, C99 to C79, C18 to C8, C100 to C80, C101 to C81, C102 to C82, C103 to C83, C104 to C84, C105 to C85, C106 to C86, C107 to C87, C108 to C88, C111 to C89, C19 to C9, C112 to C90, C113 to C91, C114 to C92, C115 to C93, C116 to C94, C117 to C95, C118 to C96, C119 to C97, C120 to C98, C121 to C99, R11 to R1, R22 to R10, R25 to R11, R26 to R12, R27 to R13, R28 to R14, R29 to R15, R30 to R16, R31 to R17, R32 to R18, R33 to R19, R12 to R2, R34 to R20, R35 to R21, R36 to R22, R37 to R23, R38 to R24, R39 to R25, R40 to R26, R41 to R27, R42 to R28, R45 to R29, R13 to R3, R46 to R30, R47 to R31, R48 to R32, R49 to R33, R50 to R34, R51 to R35, R54 to R36, R55 to R37, R56 to R38, R57 to R39, R16 to R4, R58 to R40, R59 to R41, R60 to R42, R61 to R43, R62 to R44, R63 to R45, R64 to R46, R65 to R47, R66 to R48, R67 to R49, R17 to R5, R68 to R50, R69 to R51, R70 to R52, R71 to R53, R72 to R54, R73 to R55, R74 to R56, R77 to R57, R78 to R58, R79 to R59, R18 to R6, R80 to R60, R81 to R61, R82 to R62, R85 to R63, R86 to R64, R87 to R65, R88 to R66, R89 to R67, R90 to R68, R91 to R69, R19 to R7, R92 to R70, R93 to R71, R94 to R72, R95 to R73, R96 to R74, R97 to R75, R98 to R76, R99 to R77, R100 to R78, R20 to R8, R21 to R9
Connections:
- net +3V3: no longer J11.1 (Pin_1)
- net +5VS1: now also J12.1 (Pin_1), J8.1 (Pin_1), J9.1 (Pin_1)
- net +5VS2: now also J10.1 (Pin_1), J11.1 (Pin_1), J13.1 (Pin_1)
- net GND: now also U4.7 (VDDUSB), J6.1
- net RF_IN: now also J6.2
- no-connect marks 20 -> 61
Other:
- note added: "YET TO CHANGE"

Commit message: tiny changes
Parts:
- removed D10, D12, D14: PESD5V0U1BB, symbol ESD_Diodes:ESD_DIODE
- removed D11, D13, D9: SLESD5Z5C, symbol ESD_Diodes:ESD_DIODE
- added D10, D12, D14: PESD5V0U1BB, symbol VECTRON_V1:ESD_DIODE
- added D11, D13, D9: SLESD5Z5C, symbol VECTRON_V1:ESD_DIODE
Connections:
- net +VUSB_FS: now also D10.2
- net +VUSB_HS: now also D9.2
- net GND: now also D10.1, D11.1, D12.1, D13.1, D14.1, D9.1
- net USB_FS_D+: now also D14.2
- net USB_FS_D-: now also D12.2
- net USB_HS_D+: now also D13.2
- net USB_HS_D-: now also D11.2
