File: Hardware/KiCAD files/VECTRON_V1.kicad_sch (KiCad schematic)
At the start: 242 parts, among them J1 Screw_01x02, J10 1X3-JST-XH, J11 1X3-JST-XH, J12 1X3-JST-XH, J13 1X3-JST-XH, J14 01x03_Pin, J15 01x04_Pin, J16 01x04_Pin, J17 1X4-JST-XH, J18 USB_C_Receptacle_USB2.0_16P, J19 USB_C_Receptacle_USB2.0_16P, J2 Screw_01x02, J3 Screw_01x02, J4 Conn_01x06_Pin, J5 1X4-JST-XH, J6 U_FL-R-SMT, J7 Micro_SD_Card, J8 1X3-JST-XH, J9 1X3-JST-XH, Q1 SIS447DN, Q2 IRLML2502, Q3 BSS123IXTSA1, U1 LIS2MDL, U10 TPS563201, U11 AMS1117-3.3, U2 BMP280, U3 ISM330DHCX, U4 NEO-6M-GPS, U5 TPS563201, U6 W25Q128JVS, U7 TPS563201, U8 STM32F407VGTx, U9 TPS563201, Y1 25MHz, Y2 32.678KHz

Commit message: final changes
Parts:
- removed C1, C18, C2, C3, C33, C34, C35, C36, C37, C39, C4, C5, C55, C6, C67, C68, C69, C7, C70, C71, C73, C74, C75, C80, C81, C82, C83, C84, C86, C87, C88, C89, C9: 10uf, symbol Device:C
- removed C19, C32, C38, C56, C64, C72, C79, C85, C90, C98, C99: 100nf, symbol Device:C
- removed C65: 2u2f, symbol Device:C
- removed C93, C96: 100nf, Capacitor_SMD:C_0603_1608Metric, symbol Device:C
- removed C94, C95: 10uf, Capacitor_SMD:C_0603_1608Metric, symbol Device:C
- removed D1: SS24-SMB, symbol Device:D_Schottky
- removed D11, D13: SLESD5Z5C, symbol VECTRON_V1:ESD_DIODE
- removed D14: PESD5V0U1BB, symbol VECTRON_V1:ESD_DIODE
- removed D7: white, LED_SMD:LED_0603_1608Metric, symbol Device:LED
- removed J10, J11, J12, J13, J8, J9: 1X3-JST-XH, Connector_JST:JST_XH_B3B-XH-A_1x03_P2.50mm_Vertical, symbol Connector:Conn_01x03_Pin
- removed J17: 1X4-JST-XH, symbol Connector:Conn_01x04_Pin
- removed J18: USB_C_Receptacle_USB2.0_16P, symbol Connector:USB_C_Receptacle_USB2.0_16P
- removed J6: U_FL-R-SMT, SparkFun-Connector:RP-SMA_Edge, symbol dk_Coaxial-Connectors-RF:U_FL-R-SMT_10_
- removed JP5, JP6: Jumper, Jumper:SolderJumper-2_P1.3mm_Open_RoundedPad1.0x1.5mm, symbol Jumper:SolderJumper_2_Open
- removed L1, L4, L5: SWPA5040S3R3NT 3u3h, Inductor_SMD:L_Sunlord_SWPA5040S, symbol Device:L
- removed Q1: SIS447DN, symbol Simulation_SPICE:PMOS
- removed Q2: IRLML2502, symbol Simulation_SPICE:NMOS
- removed Q3: BSS123IXTSA1, Package_TO_SOT_SMD:SOT-23, symbol Transistor_FET:BSS123
- removed R10, R21, R24, R25, R26, R53, R61, R8, R9: 10k, symbol Device:R
- removed R11, R13, R16, R17, R18, R28, R32, R33, R36, R46, R48, R51, R52: 10Ω, symbol Device:R_Small
- removed R20, R50, R58: 54k9, symbol Device:R
- removed R22, R23: 10M, symbol Device:R
- removed R49, R57, R66, R69: 5k1, symbol Device:R
- removed R55: 2k2, symbol Device:R
- removed R56: 330, symbol Device:R
- removed R63, R68: 0Ω, symbol Device:R_Small
- removed R64: 560, symbol Device:R
- removed R72, R75: 22Ω, symbol Device:R
- removed R77, R78: 100k, symbol Device:R
- removed U10, U5, U9: TPS563201, Package_TO_SOT_SMD:SOT-23-6, symbol VECTRON_V1:TPS563201
- removed U11: AMS1117-3.3, Package_TO_SOT_SMD:SOT-223-3_TabPin2, symbol Regulator_Linear:AMS1117-3.3
- added C30: 27pf, Capacitor_SMD:C_0402_1005Metric, symbol Device:C
- added C31: 15pf, Capacitor_SMD:C_0402_1005Metric, symbol Device:C
- added C42, C43, C44, C45, C46, C47: 10uf, Capacitor_SMD:C_0603_1608Metric, symbol Device:C
- added C54: 2u2f, Capacitor_SMD:C_0402_1005Metric, symbol Device:C
- added D4: 1N4148W, Diode_SMD:D_SOD-123, symbol Diode:1N4148W
- added D8: white, LED_SMD:LED_0603_1608Metric, symbol Device:LED
- added H1, H2, H3, H4: Mount_Hole, MountingHole:MountingHole_3.2mm_M3_Pad_Via, symbol Mechanical:MountingHole_Pad
- added J10, J11, J12, J13, J14, J9: Screw_01x03, TerminalBlock:TerminalBlock_Xinya_XY308-2.54-3P_1x03_P2.54mm_Horizontal, symbol Connector:Screw_Terminal_01x03
- added J18: 01x04_Pin, Connector_PinHeader_2.54mm:PinHeader_1x04_P2.54mm_Vertical, symbol Connector:Conn_01x04_Pin
- added J4: Screw_01x02, TerminalBlock_RND:TerminalBlock_RND_205-00045_1x02_P5.00mm_Horizontal, symbol Connector:Screw_Terminal_01x02
- added J7: U_FL-R-SMT_10_, digikey-footprints:Coax_Conn_U.FL, symbol dk_Coaxial-Connectors-RF:U_FL-R-SMT_10_
- added L3: SWPA5040S3R3NT 3u3h, Inductor_SMD:L_Sunlord_SWPA5040S, symbol Device:L
- added Q1: SiS447DN, Package_SO:Vishay_PowerPAK_1212-8_Single, symbol Transistor_FET:SiS443DN
- added Q2: IRLML2502TRPBF, Package_TO_SOT_SMD:TSOT-23, symbol dk_Transistors-FETs-MOSFETs-Single:IRLML2502TRPBF
- added R15: 10k, Resistor_SMD:R_0603_1608Metric, symbol Device:R
- added R17: 5k1, Resistor_SMD:R_0603_1608Metric, symbol Device:R
- added R18: 54k9, Resistor_SMD:R_0603_1608Metric, symbol Device:R
- added R42: 0Ω, Resistor_SMD:R_0603_1608Metric, symbol Device:R_Small
- added R48: 560, Resistor_SMD:R_0603_1608Metric, symbol Device:R
- added U7: TPS563201, Package_TO_SOT_SMD:SOT-23-6, symbol VECTRON_V1:TPS563201
- BT1: footprint (none) -> Battery:BatteryHolder_Multicomp_BC-2001_1x2032_1
- BZ1: footprint Buzzer_Beeper:MagneticBuzzer_PUI_AT-0927-TT-6-R -> Buzzer_Beeper:MagneticBuzzer_CUI_CMT-8504-100-SMT
- C1: renamed from C8; footprint (none) -> Capacitor_SMD:C_0603_1608Metric
- C10: renamed from C20; footprint (none) -> Capacitor_SMD:C_0603_1608Metric
- C11: renamed from C21; footprint (none) -> Capacitor_SMD:C_0603_1608Metric
- C12: renamed from C22; footprint (none) -> Capacitor_SMD:C_0603_1608Metric
- C13: renamed from C23; footprint (none) -> Capacitor_SMD:C_0603_1608Metric
- C14: renamed from C24; footprint (none) -> Capacitor_SMD:C_0603_1608Metric
- C15: renamed from C25; footprint (none) -> Capacitor_SMD:C_0603_1608Metric
- C16: renamed from C26; footprint (none) -> Capacitor_SMD:C_0603_1608Metric
- C17: renamed from C27; footprint (none) -> Capacitor_SMD:C_0603_1608Metric
- C18: renamed from C28; footprint (none) -> Capacitor_SMD:C_0603_1608Metric
- C19: renamed from C29; footprint (none) -> Capacitor_SMD:C_0603_1608Metric
- C2: renamed from C10; footprint (none) -> Capacitor_SMD:C_0603_1608Metric
- C21: renamed from C31; footprint (none) -> Capacitor_SMD:C_0603_1608Metric
- C22: renamed from C50; footprint (none) -> Capacitor_SMD:C_0603_1608Metric
- C23: renamed from C57; footprint (none) -> Capacitor_SMD:C_0603_1608Metric
- C24: renamed from C58; footprint (none) -> Capacitor_SMD:C_0603_1608Metric
- C25: renamed from C59; footprint (none) -> Capacitor_SMD:C_0603_1608Metric
- C26: renamed from C51; footprint (none) -> Capacitor_SMD:C_0603_1608Metric
- C27: renamed from C52; footprint (none) -> Capacitor_SMD:C_0603_1608Metric
- C28: renamed from C53; footprint (none) -> Capacitor_SMD:C_0603_1608Metric
- C29: renamed from C54; footprint (none) -> Capacitor_SMD:C_0603_1608Metric
- C3: renamed from C11; footprint (none) -> Capacitor_SMD:C_0603_1608Metric
- C33: renamed from C43; footprint (none) -> Capacitor_SMD:C_0603_1608Metric
- C34: renamed from C44; value 10pf -> 33pf; footprint (none) -> Capacitor_SMD:C_0402_1005Metric
- C35: renamed from C45; value 10pf -> 22pf; footprint (none) -> Capacitor_SMD:C_0402_1005Metric
- C36: renamed from C46; value 10pf -> 18pf; footprint (none) -> Capacitor_SMD:C_0402_1005Metric
- C37: renamed from C47; value 10pf -> 11pf; footprint (none) -> Capacitor_SMD:C_0402_1005Metric
- C39: renamed from C49; footprint (none) -> Capacitor_SMD:C_0603_1608Metric
- C4: renamed from C12; footprint (none) -> Capacitor_SMD:C_0603_1608Metric
- C40: value 10uf -> 100nf; footprint (none) -> Capacitor_SMD:C_0603_1608Metric
- C41: footprint (none) -> Capacitor_SMD:C_0603_1608Metric
- C48: renamed from C97; footprint (none) -> Capacitor_SMD:C_0603_1608Metric
- C49: renamed from C60; footprint (none) -> Capacitor_SMD:C_0603_1608Metric
- C5: renamed from C13; footprint (none) -> Capacitor_SMD:C_0603_1608Metric
- C50: renamed from C63; footprint (none) -> Capacitor_SMD:C_0603_1608Metric
- C51: renamed from C61; footprint (none) -> Capacitor_SMD:C_0603_1608Metric
- C52: renamed from C62; footprint (none) -> Capacitor_SMD:C_0603_1608Metric
- C55: renamed from C66; footprint (none) -> Capacitor_SMD:C_0402_1005Metric
- C6: renamed from C14; footprint (none) -> Capacitor_SMD:C_0603_1608Metric
- C66: renamed from C77; footprint (none) -> Capacitor_SMD:C_0603_1608Metric
- C67: renamed from C78; footprint (none) -> Capacitor_SMD:C_0603_1608Metric
- C7: renamed from C15; footprint (none) -> Capacitor_SMD:C_0603_1608Metric
- C78: renamed from C91; footprint (none) -> Capacitor_SMD:C_0603_1608Metric
- C79: renamed from C92; footprint (none) -> Capacitor_SMD:C_0603_1608Metric
- C8: renamed from C16; footprint (none) -> Capacitor_SMD:C_0603_1608Metric
- C9: renamed from C17; footprint (none) -> Capacitor_SMD:C_0603_1608Metric
- D1: renamed from D2; value SS24-SMB -> SS24B-Slkor; footprint (none) -> Diode_SMD:D_SMA
- D10: renamed from D12; footprint (none) -> Diode_SMD:D_SOD-523
- D11: renamed from D9; footprint (none) -> Diode_SMD:D_SOD-523
- D2: renamed from D3; footprint (none) -> Diode_SMD:D_SOD-523
- D9: renamed from D10; footprint (none) -> Diode_SMD:D_SOD-523
- FB1: footprint (none) -> Inductor_SMD:L_0603_1608Metric
- J1: renamed from J2; footprint (none) -> TerminalBlock:TerminalBlock_Xinya_XY308-2.54-2P_1x02_P2.54mm_Horizontal
- J15: renamed from J14; footprint (none) -> Connector_PinHeader_2.54mm:PinHeader_1x03_P2.54mm_Vertical
- J16: renamed from J15; footprint (none) -> Connector_PinHeader_2.54mm:PinHeader_1x04_P2.54mm_Vertical
- J17: renamed from J16; footprint (none) -> Connector_PinHeader_2.54mm:PinHeader_1x04_P2.54mm_Vertical
- J19: footprint (none) -> Connector_USB:USB_C_Receptacle_GCT_USB4105-xx-A_16P_TopMnt_Horizontal
- J2: renamed from J1; footprint (none) -> TerminalBlock_RND:TerminalBlock_RND_205-00045_1x02_P5.00mm_Horizontal
- J3: footprint (none) -> TerminalBlock:TerminalBlock_Xinya_XY308-2.54-2P_1x02_P2.54mm_Horizontal
- J5: renamed from J4; value Conn_01x06_Pin -> 01x06_Pin; footprint (none) -> Connector_PinHeader_2.54mm:PinHeader_1x06_P2.54mm_Vertical
- J6: renamed from J5; value 1X4-JST-XH -> 01x04_Pin; footprint (none) -> Connector_PinHeader_2.54mm:PinHeader_1x04_P2.54mm_Vertical
- J8: renamed from J7; footprint (none) -> Connector_Card:microSD_HC_Molex_47219-2001
- L2: value 27nh -> 27uh; footprint Inductor_SMD:L_0402_1005Metric -> Inductor_SMD:L_0805_2012Metric
- R1, R2, R3, R4, R5, R6, R7: footprint (none) -> Resistor_SMD:R_0603_1608Metric
- R10: renamed from R15; footprint (none) -> Resistor_SMD:R_0603_1608Metric
- R11: renamed from R30; footprint (none) -> Resistor_SMD:R_0603_1608Metric
- R12: renamed from R31; footprint (none) -> Resistor_SMD:R_0603_1608Metric
- R13: renamed from R34; footprint (none) -> Resistor_SMD:R_0603_1608Metric
- R14: renamed from R27; footprint (none) -> Resistor_SMD:R_0603_1608Metric
- R16: renamed from R29; footprint (none) -> Resistor_SMD:R_0805_2012Metric
- R19: value 5k1 -> 10k; footprint (none) -> Resistor_SMD:R_0603_1608Metric
- R20: renamed from R35; footprint (none) -> Resistor_SMD:R_0603_1608Metric
- R21: renamed from R37; footprint (none) -> Resistor_SMD:R_0603_1608Metric
- R22: renamed from R38; footprint (none) -> Resistor_SMD:R_0603_1608Metric
- R23: renamed from R39; footprint (none) -> Resistor_SMD:R_0603_1608Metric
- R24: renamed from R40; footprint (none) -> Resistor_SMD:R_0603_1608Metric
- R25: renamed from R41; footprint (none) -> Resistor_SMD:R_0603_1608Metric
- R26: renamed from R42; footprint (none) -> Resistor_SMD:R_0603_1608Metric
- R27: renamed from R43; footprint (none) -> Resistor_SMD:R_0603_1608Metric
- R28: renamed from R44; footprint (none) -> Resistor_SMD:R_0603_1608Metric
- R29: renamed from R47; footprint (none) -> Resistor_SMD:R_0603_1608Metric
- R33: renamed from R54; value 1k -> 360; footprint (none) -> Resistor_SMD:R_0603_1608Metric
- R36: renamed from R59; value 2k2 -> 4k7; footprint (none) -> Resistor_SMD:R_0603_1608Metric
- R37: renamed from R60; footprint (none) -> Resistor_SMD:R_0603_1608Metric
- R39: renamed from R62; footprint (none) -> Resistor_SMD:R_0603_1608Metric
- R40: renamed from R65; value 18k -> 30k; footprint (none) -> Resistor_SMD:R_0603_1608Metric
- R41: renamed from R74; footprint (none) -> Resistor_SMD:R_0603_1608Metric
- R43: renamed from R67; footprint (none) -> Resistor_SMD:R_0603_1608Metric
- R44: renamed from R70; footprint (none) -> Resistor_SMD:R_0603_1608Metric
- R45: value 10Ω -> 0Ω; footprint (none) -> Resistor_SMD:R_0603_1608Metric
- R46: renamed from R71; footprint (none) -> Resistor_SMD:R_0603_1608Metric
- R47: renamed from R73; value 22Ω -> 27Ω; footprint (none) -> Resistor_SMD:R_0603_1608Metric
- R49: renamed from R76; footprint (none) -> Resistor_SMD:R_0603_1608Metric
- R8: renamed from R12; footprint (none) -> Resistor_SMD:R_0603_1608Metric
- R9: renamed from R14; footprint (none) -> Resistor_SMD:R_0603_1608Metric
- S1, S2: footprint digikey-footprints:Switch_Tactile_THT_B3F-1xxx -> TSA017A2518B:TSA017A2518B
- Y1: value 25MHz -> YSX321SL-25MHz; footprint (none) -> Crystal:Crystal_SMD_3225-4Pin_3.2x2.5mm
- Y2: value 32.678KHz -> YXC-Y-26; footprint (none) -> Crystal:Crystal_DS26_D2.0mm_L6.0mm_Horizontal
- renumbered C30 to C20, C42 to C32, C48 to C38, C76 to C65, D4 to D3, D8 to D7, L3 to L1, U2 to U1, U1 to U2, U7 to U5
Connections:
- net +VUSB_HS is gone; now on net USB_FS_D+: D11.2
- net SHIELD_FS is gone; now on net GND: J19.S1 (SHIELD)
- net +3V3: now also C67.2, D6.4 (VDD), D4.1 (K)
- net +5V: now also C44.2, C45.2, C46.2, C47.2, J18.4 (Pin_4), L3.2, R18.1, R48.1; no longer C67.2, D6.4 (VDD)
- net +MAIN_BATT: now also J2.1 (Pin_1), Q1.5 (D); no longer J2.2 (Pin_2)
- net +VCOM: now also C42.2, C43.2, Q1.1 (S), Q1.2 (S), Q1.3 (S), R17.1, U7.3 (VIN); no longer C40.2, R19.1
- net 5VLED: now also D8.2 (A), R48.2
- net BUZZ_GATE: now also Q2.1 (G)
- net EN5: now also R17.2, U7.5 (EN); no longer R19.2
- net FLASH_CS: now also U8.29 (PA4)
- net GND: now also J2.2 (Pin_2), R19.2, C42.1, C43.1, C44.1, C45.1, C46.1, C47.1, C54.1, D8.1 (K), H1.1, H2.1, H3.1, H4.1, J10.3 (Pin_3), J11.3 (Pin_3), J12.3 (Pin_3), J13.3 (Pin_3), J14.3 (Pin_3), J18.2 (Pin_2), J4.1 (Pin_1), J7.1, J9.3 (Pin_3), Q2.2 (S), R15.1, U7.1 (GND); no longer C40.1, J2.1 (Pin_1)
- net HSE_IN: now also Y1.1; no longer Y1.3
- net HSE_OUT: now also Y1.3; no longer Y1.1
- net IMU_CS: now also U8.33 (PC4)
- net IMU_INT1: now also U3.4 (INT1), U8.40 (PE9); no longer U8.3 (PE4)
- net IMU_INT2: now also U3.9 (INT2), U8.41 (PE10); no longer U8.4 (PE5)
- net LSE_IN: now also Y2.2; no longer Y2.1
- net LSE_OUT: now also Y2.1; no longer Y2.2
- net PROG_LED: now also D6.3 (DIN)
- net RECOV_1: now also J13.2 (Pin_2)
- net RECOV_2: now also J14.2 (Pin_2)
- net RF_IN: now also J7.2
- net SDIO_CK: now also U8.80 (PC12)
- net SDIO_CMD: now also U8.83 (PD2)
- net SDIO_D0: now also U8.65 (PC8); no longer R45.2
- net SDIO_D1: now also U8.66 (PC9)
- net SDIO_D2: now also U8.78 (PC10)
- net SDIO_D3: now also U8.79 (PC11)
- net SERVO_X1: now also J9.2 (Pin_2)
- net SERVO_X2: now also J10.2 (Pin_2)
- net SERVO_Y1: now also J11.2 (Pin_2)
- net SERVO_Y2: now also J12.2 (Pin_2)
- net SPI1_MISO: now also U3.1 (SDO/SA0)
- net SPI1_MOSI: now also U8.32 (PA7)
- net SPI1_SCK: now also U8.30 (PA5)
- net SPI2_MISO: now also J17.4 (Pin_4), U6.2 (DO/IO_{1}); no longer J17.3 (Pin_3)
- net SPI2_MOSI: now also J17.3 (Pin_3), U8.18 (PC3); no longer J17.4 (Pin_4)
- net SPI2_SCK: now also U8.47 (PB10)
- net SW5: now also C40.2, L3.1, U7.2 (SW)
- net USART1_RX: now also R10.1; no longer R8.1
- net USART1_TX: now also R8.1; no longer R10.1
- net USART2_RX: now also J18.3 (Pin_3)
- net USART2_TX: now also J18.1 (Pin_1)
- net VBST5: now also C40.1, U7.6 (VBST)
- net VCAP_1: now also C54.2
- net VFB5: now also R19.1, R18.2, U7.4 (VFB)
- net SDIO_DECT: now reaches U8.43 (PE12)
- net SDIO_DECT: now also R15.2
- net at R45.1: no longer U8.65 (PC8)
- net at BZ1.2 (-): now also D4.2 (A), Q2.3 (D)
- net at D2.2 (A), R4.2: now also Q1.4 (G)
- net HS_D+: no longer names the net of U8.54 (PB15)
- net HS_D-: no longer names the net of U8.53 (PB14)
- net gps_inductor renamed GPS_INDUCTOR
- new net +6V: J10.1 (Pin_1), J11.1 (Pin_1), J12.1 (Pin_1), J13.1 (Pin_1), J14.1 (Pin_1), J4.2 (Pin_2), J9.1 (Pin_1)
- no-connect marks 61 -> 64
Other:
- note added: "6V SERVO"
- note added: "MOUNTING HOLES"
- note removed: "3V3 LDO (REDUNDANT)"
- note removed: "3V3 pwr flag is not required as AMS1117 marks 3V3 pin as power output"
- note removed: "USB TYPE C HIGH SPEED"
- note removed: "XY117B-3.81"
- note removed: "YET TO CHANGE"
- moved on the sheet: BT1, C1, C10, C16, C18, C19, C22, C23, C24, C25, C26, C27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
